File: MIDI-PCB/MIDI-PCB.kicad_sch (KiCad schematic)
At the start: 43 parts, among them J1 display, J2 Keypad, J3 Rotary encoder, J4 Conn_01x06, J5 Conn_01x06, J6 Conn_01x06, J7 Conn_01x12, J8 Conn_01x12, J9 Conn_01x12, SW1 SW_Push, SW2 SW_Push, U1 XIAO-RP2040-SMD

Commit message: YAY
Connections:
- net at D2.1 (DOUT): now also D5.3 (DIN)
Changed lines of the file:
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@@
+	(wire
+		(pts
+			(xy 82.55 135.89) (xy 90.17 135.89)
+		)
+		(stroke
+			(width 0)
+			(type default)
+		)
+	)
 	(wire
 		(pts
